File: crispy-keyboard.sch (KiCad schematic (older format))
At the start: 169 parts, among them J1 Conn_01x03_Female, J2 Conn_01x02, SW1 KEYSW, SW10 KEYSW, SW11 KEYSW, SW12 KEYSW, SW13 KEYSW, SW14 KEYSW, SW15 KEYSW, SW16 KEYSW, SW17 KEYSW, SW18 KEYSW, SW19 KEYSW, SW2 KEYSW, SW20 KEYSW, SW21 KEYSW, SW22 KEYSW, SW23 KEYSW, SW24 KEYSW, SW25 KEYSW, SW26 KEYSW, SW27 KEYSW, SW28 KEYSW, SW29 KEYSW, SW3 KEYSW, SW30 KEYSW, SW31 KEYSW, SW32 KEYSW, SW33 KEYSW, SW34 KEYSW, SW35 KEYSW, SW36 KEYSW, SW37 KEYSW, SW38 KEYSW, SW39 KEYSW, SW4 KEYSW, SW40 KEYSW, SW41 KEYSW, SW42 KEYSW, SW43 KEYSW, SW44 KEYSW, SW45 KEYSW, SW46 KEYSW, SW47 KEYSW, SW48 KEYSW, SW49 KEYSW, SW5 KEYSW, SW50 KEYSW, SW51 KEYSW, SW52 KEYSW, SW53 KEYSW, SW54 KEYSW, SW55 KEYSW, SW56 KEYSW, SW57 KEYSW, SW58 KEYSW, SW59 KEYSW, SW6 KEYSW, SW60 KEYSW, SW61 KEYSW, SW62 KEYSW, SW63 KEYSW, SW64 KEYSW, SW65 KEYSW, SW66 KEYSW, SW67 KEYSW, SW68 KEYSW, SW69 KEYSW, SW7 KEYSW, SW70 KEYSW, SW71 KEYSW, SW72 KEYSW, SW73 KEYSW, SW74 KEYSW, SW75 KEYSW, SW76 KEYSW, SW77 KEYSW, SW78 KEYSW, SW79 KEYSW, SW8 KEYSW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

Commit message: Added BlueMacro PCB. Added Plate PCB.
Parts:
- added SW85: Bat, crispy-keyboard:CK_Switches-L101011ML04Q-0-0-MFG, symbol Switch:SW_Push
- J1: value Conn_01x03_Female -> RGB Strip
- J2: value Conn_01x02 -> Battery
- LD2: value LED -> Power
- LD3: value LED -> Bluetooth
- SW83: value Rotary_Encoder_Switch -> Rotary Encoder
- SW84: value SW_Push -> Reset
Connections:
- net at J2.1 (Pin_1): now also SW85.2; no longer U1.32 (VBatt)
- new net: SW85.1, U1.32 (VBatt)
Changed lines of the file:
@@
 P 6040 8613
 F 0 "LD2" H 6033 8830 50  0000 C CNN
-F 1 "LED" H 6033 8739 50  0000 C CNN
+F 1 "Power" H 6033 8739 50  0000 C CNN
 F 2 "crispy-keyboard:LED_D3.0mm" H 6040 8613 50  0001 C CNN
 F 3 "~" H 6040 8613 50  0001 C CNN
@@
 P 6034 9117
 F 0 "LD3" H 6027 9334 50  0000 C CNN
-F 1 "LED" H 6027 9243 50  0000 C CNN
+F 1 "Bluetooth" H 6027 9243 50  0000 C CNN
 F 2 "crispy-keyboard:LED_D3.0mm" H 6034 9117 50  0001 C CNN
 F 3 "~" H 6034 9117 50  0001 C CNN
@@
 P 7368 8615
 F 0 "SW84" H 7368 8900 50  0000 C CNN
-F 1 "SW_Push" H 7368 8809 50  0000 C CNN
+F 1 "Reset" H 7368 8809 50  0000 C CNN
 F 2 "crispy-keyboard:SW_PUSH_6mm" H 7368 8815 50  0001 C CNN
 F 3 "~" H 7368 8815 50  0001 C CNN
@@
 P 7705 9054
 F 0 "J1" V 7643 8866 50  0000 R CNN
-F 1 "Conn_01x03_Female" V 7552 8866 50  0000 R CNN
+F 1 "RGB Strip" V 7552 8866 50  0000 R CNN
 F 2 "Connector_PinHeader_2.00mm:PinHeader_1x03_P2.00mm_Horizontal" H 7705 9054 50  0001 C CNN
 F 3 "~" H 7705 9054 50  0001 C CNN
@@
 P 4178 7633
 F 0 "J2" H 4096 7850 50  0000 C CNN
-F 1 "Conn_01x02" H 4096 7759 50  0000 C CNN
+F 1 "Battery" H 4096 7759 28  0000 C CNN
 F 2 "Connector_PinHeader_2.54mm:PinHeader_1x02_P2.54mm_Vertical" H 4178 7633 50  0001 C CNN
 F 3 "~" H 4178 7633 50  0001 C CNN
@@
 $EndComp
 Wire Wire Line
-	5342 7597 4378 7597
+	5342 7597 4830 7597
 Wire Wire Line
 	4378 7597 4378 7633
@@
 P 7123 6947
 F 0 "SW83" H 7123 7314 50  0000 C CNN
-F 1 "Rotary_Encoder_Switch" H 7123 7223 50  0000 C CNN
+F 1 "Rotary Encoder" H 7123 7223 50  0000 C CNN
 F 2 "crispy-keyboard:Bourns-PEC11R-4120F-S0018-MFG" H 6973 7107 50  0001 C CNN
 F 3 "~" H 7123 7207 50  0001 C CNN
@@
 Text GLabel 6628 8613 2    50   Input ~ 0
 Red_LED
+$Comp
+L Switch:SW_Push SW85
+U 1 1 60BF97C5
+P 4630 7597
+F 0 "SW85" H 4630 7882 50  0000 C CNN
+F 1 "Bat" H 4630 7791 50  0000 C CNN
+F 2 "crispy-keyboard:CK_Switches-L101011ML04Q-0-0-MFG" H 4630 7797 50  0001 C CNN
+F 3 "~" H 4630 7797 50  0001 C CNN
+	1    4630 7597
+	-1   0    0    -1
+$EndComp
+Wire Wire Line
+	4430 7597 4378 7597
 $EndSCHEMATC
