File: crispy-keyboard.kicad_pcb (KiCad board)
At the start: 2 copper layers, 330 x 120.8 mm, 184 parts, among them J1 Conn_01x03_Female, J2 Conn_01x02, SW1 KEYSW, SW10 KEYSW, SW11 KEYSW, SW12 KEYSW, SW13 KEYSW, SW14 KEYSW, SW15 KEYSW, SW16 KEYSW, SW17 KEYSW, SW18 KEYSW, SW19 KEYSW, SW2 KEYSW, SW20 KEYSW, SW21 KEYSW, SW22 KEYSW, SW23 KEYSW, SW24 KEYSW, SW25 KEYSW, SW26 KEYSW, SW27 KEYSW, SW28 KEYSW, SW29 KEYSW, SW3 KEYSW, SW30 KEYSW, SW31 KEYSW, SW32 KEYSW, SW33 KEYSW, SW34 KEYSW, SW35 KEYSW, SW36 KEYSW, SW37 KEYSW, SW38 KEYSW, SW39 KEYSW, SW4 KEYSW, SW40 KEYSW, SW41 KEYSW, SW42 KEYSW, SW43 KEYSW, SW44 KEYSW, SW45 KEYSW, SW46 KEYSW, SW47 KEYSW, SW48 KEYSW, SW49 KEYSW, SW5 KEYSW, SW50 KEYSW, SW51 KEYSW, SW52 KEYSW, SW53 KEYSW, SW54 KEYSW, SW55 KEYSW, SW56 KEYSW, SW57 KEYSW, SW58 KEYSW, SW59 KEYSW, SW6 KEYSW, SW60 KEYSW, SW61 KEYSW, SW62 KEYSW, SW63 KEYSW, SW64 KEYSW, SW65 KEYSW, SW66 KEYSW, SW67 KEYSW, SW68 KEYSW, SW69 KEYSW, SW7 KEYSW, SW70 KEYSW, SW71 KEYSW, SW72 KEYSW, SW73 KEYSW, SW74 KEYSW, SW75 KEYSW, SW76 KEYSW, SW77 KEYSW, SW78 KEYSW, SW79 KEYSW, SW8 KEYSW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

Commit message: Shifted macro footprint for better usb access. Shifted rotary encoder footprint for better access
Parts:
- removed the REF** at (32.6, 63.6)
- added REF**: MountingHole_2.2mm_M2_Pad, crispy-keyboard:MountingHole_2.2mm_M2_Pad, F.Cu at (38.1, 161.4)
- added REF**: MountingHole_2.2mm_M2_Pad, crispy-keyboard:MountingHole_2.2mm_M2_Pad, F.Cu at (33.0, 63.6)
- moved J2 1.77 mm to (329.9, 77.6)
- moved J1 1.77 mm to (335.5, 75.8)
- moved U1 1.77 mm to (315.8, 72.8)
- moved REF** 1.08 mm to (33.0, 81.6)
- moved REF** 1.00 mm to (354.8, 81.6)
- moved SW82 0.37 mm to (41.3, 165.9)
- moved SW79 0.37 mm to (41.3, 108.7)
- moved SW81 0.37 mm to (41.3, 146.8)
- moved SW80 0.37 mm to (41.3, 127.8)
- renumbered LD3 to Bluetooth, LD2 to Power
Routing:
- net Net-(D62-Pad2): track 367.2 -> 523.5 mm
- net col10: track 242.4 -> 182.8 mm
- net GND: track 549.9 -> 587.7 mm, vias 54 -> 56
- net col12: track 177.8 -> 170.8 mm
- net row4: track 399.4 -> 394.9 mm
- net col14: track 96.4 -> 92.4 mm
- net col3: track 449.4 -> 447.1 mm
- net Net-(D43-Pad2): track 164.9 -> 166.7 mm
- net Net-(D29-Pad2): track 139.2 -> 141.0 mm
- net Net-(D66-Pad2): track 202.2 -> 203.9 mm
- net Net-(D68-Pad2): track 244.2 -> 246.0 mm
- net Net-(D65-Pad2): track 226.7 -> 228.5 mm
- net Net-(D77-Pad2): track 47.7 -> 46.0 mm
- net Net-(LD1-Pad2): track 450.6 -> 448.9 mm
- net col9: track 251.0 -> 249.6 mm
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Other:
- board size 330 x 120.8 mm -> 329.6 x 120.8 mm

Commit message: Added BlueMacro PCB. Added Plate PCB.
Parts:
- added SW85: Bat, crispy-keyboard:CK_Switches-L101011ML04Q-0-0-MFG, B.Cu at (318.0, 64.6)
- Bluetooth: value LED -> Bluetooth
- J1: value Conn_01x03_Female -> RGB Strip
- J2: value Conn_01x02 -> Battery
- Power: value LED -> Power
- SW83: value Rotary_Encoder_Switch -> Rotary Encoder
- moved J2 0.13 mm to (329.8, 77.7)
Connections:
- U1 pad 32: Net-(J2-Pad1) -> Net-(SW85-Pad1)
Routing:
- net col10: track 182.8 -> 241.9 mm
- net Net-(J2-Pad1): track 26.8 -> 15.7 mm, vias 2 -> 0
- net col12: track 170.8 -> 178.3 mm
- net Net-(SW85-Pad1): track 0.00 -> 6.49 mm
- net col9: track 249.6 -> 251.4 mm
- net col8: track 236.1 -> 237.9 mm
- net col6: track 301.7 -> 303.4 mm
- net col11: track 203.3 -> 205.1 mm
- net Net-(LD1-Pad2): track 448.9 -> 450.7 mm
- net col13: track 156.7 -> 158.4 mm
- net col7: track 255.4 -> 257.2 mm
- net row2: track 312.9 -> 311.6 mm
- net row3: track 432.1 -> 430.8 mm
- net row0: track 301.7 -> 302.9 mm
- net RESET: track 117.1 -> 116.1 mm
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Other:
- board text added: "5V"
- board text added: "Data"
- board text added: "GND"
