File: plate/discipline-pcb.kicad_pcb (KiCad board)
At the start: 2 copper layers, 329.9 x 96.2 mm, 0 parts

Commit message: Finished plate
Parts:
- added G***: LOGO, crispy-keyboard:crispy_logo, F.Cu at (52.3, 169.1)
Other:
- board size 329.9 x 96.2 mm -> 330.1 x 96.2 mm

Commit message: Finished Plate. Fixed errors (missing via, missing solder mask) on BlueMacro
Parts:
- removed G***: LOGO, crispy-keyboard:crispy_logo
Other:
- outline, holes or cut-outs redrawn
